File: KICAD/SHIELD_GAS.kicad_sch (KiCad schematic)
At the start: 24 parts, among them J1 Conn_01x08_Female, J2 Conn_01x04_Male, Q1 Q_NPN_BCE, SW1 SW_SPDT, U1 ESP32-DEVKITC-32D, U2 TO_5, U3 LTC1050CN8, U4 TL071

Commit message: update
Connections:
- net 3V3: now also R6.2, R7.1; no longer R1.1, R3.1
- net GND: now also R1.2, R9.1; no longer R5.2, R7.2
- net Isens: now also R5.1; no longer R6.1
- net R_ALU: now also R6.1; no longer R3.2
- net at C2.1, U3.2 (-IN): now also R2.1, R3.1; no longer R8.1, R9.1
- net at Q1.1 (B), R4.1: now also R9.2; no longer R5.1
- net at C1.1, U3.3 (+IN): now also R1.1, R5.2; no longer R6.2, R7.1
- net at C2.2, R10.1, U3.6 (OUT): now also R3.2; no longer R9.2
- new net: R7.2, R8.1, U4.3 (+)
Other:
- moved on the sheet: C3, R1, R2, R3, R5, R6, R7, R8, R9, SW1
